File: counter/counter.sch (KiCad schematic (older format))
At the start: 16 parts, among them U1 sohamsen_synchronous_down_cou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, U2 adc_bridge_2, U3 plot_v1, U4 dac_bridge_3, U5 plot_v1, U6 plot_v1, U7 plot_v1

Commit message: edited counter
Parts:
- added U8: plot_v1, symbol plot_v1
Connections:
- net RST: now reaches U2.2 (IN2), v1.1 (+)
- net RST: now also U8.~
Changed lines of the file:
@@
 	3600 4650 3600 4450
 Wire Wire Line
-	3600 4450 3950 4450
+	3200 4450 3950 4450
 Wire Wire Line
 	2550 2100 2550 2400
@@
 	4250 1350 4000 1350
 Connection ~ 4000 1350
+$Comp
+L plot_v1 U8
+U 1 1 63419ED4
+P 3400 4650
+F 0 "U8" H 3400 5150 60  0000 C CNN
+F 1 "plot_v1" H 3600 5000 60  0000 C CNN
+F 2 "" H 3400 4650 60  0000 C CNN
+F 3 "" H 3400 4650 60  0000 C CNN
+	1    3400 4650
+	1    0    0    -1
+$EndComp
+Connection ~ 3600 4450
+Text GLabel 3200 4450 0    60   Input ~ 0
+RST
+Connection ~ 3400 4450
 $EndSCHEMATC
